Commit message: Aggiornamento fra2mo_description

File: urdf/lidar_gazebo_macro.xacro (robot description, xacro)
@@ -26,5 +26,5 @@
       <parent link="${parent}" />
       <child link="laser_frame" />
-      <origin rpy="0 0 0" xyz="0.0 0.0 0.031" />
+      <origin rpy="0 0 ${-M_PI}" xyz="0.0 0.0 0.031" />
     </joint>
   </xacro:macro>
