Commit message: Aggiorna e pulisci file URDF, launch e macro; aggiungi test.urdf e fra2mo.urdf.xacro; rimuovi file obsoleti

File: urdf/d435_gazebo_macro.xacro (robot description, xacro)
@@ -1,16 +1,13 @@
 <?xml version="1.0"?>
-<robot name="d435_gazebo_macro" xmlns:xacro="http://www.ros.org/wiki/xacro">
-  <!--xacro:include filename="$(find fra2mo_description)/urdf/utility_macro.xacro" /-->
+<robot name="d435_gazebo_macro" xmlns:xacro="http://ros.org/wiki/xacro">
   <xacro:include filename="$(find realsense2_description)/urdf/_d435.urdf.xacro" />
-  <xacro:macro name="d435_gazebo_sensor" params="parent" >
+  <xacro:macro name="d435_gazebo_sensor" params="parent">
     <xacro:sensor_d435 parent="${parent}" use_nominal_extrinsics="true" add_plug="false" use_mesh="true">
-      <origin xyz="0 0 0" rpy="0 0 0"/>
+      <origin xyz="0 0 0" rpy="0 0 0" />
     </xacro:sensor_d435>
     <gazebo reference="${parent}">
-      <sensor type="rgbd_camera" name="depth_camera">
+      <sensor type="depth_camera" name="depth_camera">
         <always_on>true</always_on>
         <update_rate>30.0</update_rate>
-        <topic>depth_camera</topic>
-        <gz_frame_id>d435_link</gz_frame_id>
         <camera>
           <horizontal_fov>1.3962634</horizontal_fov>
@@ -21,14 +18,19 @@
           </image>
           <clip>
-            <near>0.1</near>
+            <near>0.01</near>
             <far>100</far>
           </clip>
-          <depth_camera>
-            <clip>
-              <near>0.1</near>
-              <far>10</far>
-            </clip>
-          </depth_camera>
         </camera>
+        <plugin name="GazeboRosDepthCamera" filename="libgazebo_ros_depth_camera.so">
+          <ros>
+            <namespace>/</namespace>
+            <remapping>~/depth/image_raw:=/depth_camera/image_raw</remapping>
+            <remapping>~/depth/camera_info:=/depth_camera/camera_info</remapping>
+            <remapping>~/points:=/depth/points</remapping>
+          </ros>
+          <update_rate>30.0</update_rate>
+          <camera_name>depth_camera</camera_name>
+          <frame_name>camera_depth_optical_frame</frame_name>
+        </plugin>
       </sensor>
     </gazebo>

File: urdf/fra2mo_base_macro.xacro (robot description, xacro)
@@ -1,159 +1,141 @@
 <?xml version="1.0"?>
-<robot name="fra2mo_base_macro" xmlns:xacro="http://www.ros.org/wiki/xacro">
+<robot  xmlns:xacro="http://www.ros.org/wiki/xacro">
   <xacro:include filename="$(find fra2mo_description)/urdf/utility_macro.xacro" />
-  <!-- Base properties -->
-	<xacro:property name="base_height" value="0.180" />
-  <xacro:property name="base_radius" value="0.11" />
-  <xacro:property name="base_mass" value="2" />
-  <xacro:property name="wheel_mass" value="0.2" />
-  <xacro:property name="wheel_radius" value="0.035" />
-  <xacro:property name="wheel_axle" value="0.124" />
   <!-- WHOLE BASE MACRO-->
   <xacro:macro name="fra2mo_base" > <!--fb : front, back ; lr: left, right -->
-      <!--Actual body/chassis of the robot-->
+    <!-- Base properties -->
+    <xacro:property name="base_height" value="0.180" />
+    <xacro:property name="base_radius" value="0.11" />
+    <xacro:property name="base_mass" value="5" />
+    <xacro:property name="wheel_mass" value="2.5" />
+    <xacro:property name="wheel_radius" value="0.035" />
+    <xacro:property name="wheel_axle" value="0.13" />
+    <!-- Actual body/chassis of the robot -->
     <link name="base_footprint">
     </link>
     <link name="base_link">
+      <!-- Inertial properties -->
       <inertial>
+        <origin xyz="0 0 0" />
         <mass value="${base_mass}" />
-        <origin xyz="0 0 -0.05" /> <!-- baricentro abbassato di 5 cm -->
-        <inertia ixx="0.01145" ixy="0.0" ixz="0.0" iyy="0.01145" iyz="0.0" izz="0.0121"/>
+        <xacro:cylinder_inertia m="${base_mass}" r="${base_radius}" h="${base_height}" />
       </inertial>
+      <!-- Visual representation -->
       <visual>
         <geometry>
-          <mesh filename="package://fra2mo_description/meshes/fra2mo_body.stl" scale="0.001 0.001 0.001 "/>
+          <mesh filename="file://$(find fra2mo_description)/meshes/fra2mo_body.stl" scale="0.001 0.001 0.001" />
         </geometry>
-        <material name="White"/>
-        <origin rpy="0 0 0" xyz="0 0 0"/>
+        <material name="Blue" />
+        <origin xyz="0 0 0" rpy="0 0 0" />
+      </visual>
+      <!-- Collision properties -->
+      <collision>
+        <geometry>
+          <cylinder length="${base_height}" radius="${base_radius}" />
+        </geometry>
+        <origin xyz="0 0.0 ${(base_height/2.0)-0.05}" rpy="0 0 0" />
+      </collision>
+      <collision>
+        <geometry>
+          <sphere radius="0.019" />
+        </geometry>
+        <origin xyz="-0.0825 0.0 -0.04" rpy="0 0 0" />
+      </collision>
+    </link>
+    <!-- Left Wheel -->
+    <link name="left_wheel_link">
+      <visual>
+        <geometry>
+          <mesh filename="file://$(find fra2mo_description)/meshes/fra2mo_wheel.stl" scale="0.001 0.001 0.001" />
+        </geometry>
+        <material name="Black" />
+        <origin xyz="0 0 0" rpy="0 0 0" />
       </visual>
       <collision>
         <geometry>
-          <cylinder length="${base_height}" radius="${base_radius}"/>
+          <mesh filename="file://$(find fra2mo_description)/meshes/fra2mo_wheel.stl" scale="0.001 0.001 0.001" />
         </geometry>
-        <origin rpy="0 0 0" xyz="0 0.0 ${(base_height/2.0)-0.05}"/>
+        <origin xyz="0 0 0" rpy="0 0 0" />
       </collision>
-      <collision>
-        <geometry>
-          <sphere radius="0.019"/>
-        </geometry>
-        <origin rpy="0 0 0" xyz="-0.0825 0.0 -0.04"/>
-      </collision>
+      <inertial>
+        <origin xyz="0 0 0" />
+        <mass value="${wheel_mass}" />
+        <inertia ixx="0.001" ixy="0.0" ixz="0.0" iyy="0.001" iyz="0.0" izz="0.001" />
+      </inertial>
     </link>
-    <link name="left_wheel_link">
+    <!-- Right Wheel -->
+    <link name="right_wheel_link">
       <visual>
         <geometry>
-          <mesh filename="package://fra2mo_description/meshes/fra2mo_wheel.stl" scale="0.001 0.001 0.001 "/>
+          <mesh filename="file://$(find fra2mo_description)/meshes/fra2mo_wheel.stl" scale="0.001 0.001 0.001" />
         </geometry>
         <material name="Black"/>
-        <origin rpy="0 0 0" xyz="0 0 0"/>
+        <origin xyz="0 0 0" rpy="0 0 0" />
       </visual>
       <collision>
         <geometry>
-          <cylinder radius="${wheel_radius}" length="0.02"/> </geometry>
-        <origin rpy="1.570796 0 0" xyz="0 0 0"/>
+          <mesh filename="file://$(find fra2mo_description)/meshes/fra2mo_wheel.stl" scale="0.001 0.001 0.001" />
+        </geometry>
+        <origin xyz="0 0 0" rpy="0 0 0" />
       </collision>
       <inertial>
-          <mass value="${wheel_mass}" />
-          <origin xyz="0 0 0" />
-          <inertia ixx="0.0000679" ixy="0.0" ixz="0.0"
-                   iyy="0.0000679" iyz="0.0"
-                   izz="0.0001225" />
+        <origin xyz="0 0 0" />
+        <mass value="${wheel_mass}" />
+        <inertia ixx="0.001" ixy="0.0" ixz="0.0" iyy="0.001" iyz="0.0" izz="0.001" />
       </inertial>
     </link>
-    <link name="right_wheel_link">
-      <visual>
-        <geometry>
-          <mesh filename="package://fra2mo_description/meshes/fra2mo_wheel.stl" scale="0.001 0.001 0.001 "/>
-        </geometry>
-        <material name="Black"/>
-        <origin rpy="0 0 0" xyz="0 0 0"/>
-      </visual>
-      <collision>
-        <geometry>
-          <cylinder radius="${wheel_radius}" length="0.02"/> </geometry>
-        <origin rpy="1.570796 0 0" xyz="0 0 0"/>
-      </collision>
-      <inertial>
-          <mass value="${wheel_mass}" />
-          <origin xyz="0 0 0" />
-          <inertia ixx="0.0000679" ixy="0.0" ixz="0.0"
-                   iyy="0.0000679" iyz="0.0"
-                   izz="0.0001225" />
-      </inertial>
-    </link>
+    <!-- Additional Links -->
     <link name="d435_link">
     </link>
-    <link name="lidar_link">
-    </link>
+    <link name="lidar_link" />
+    <!-- Joints -->
     <joint name="base_footprint_joint" type="fixed">
-      <parent link="base_footprint"/>
-      <child link="base_link"/>
-      <origin rpy="0 0 0" xyz="0.0 0.0 0.059"/>
+      <parent link="base_footprint" />
+      <child link="base_link" />
+      <origin xyz="0.0 0.0 0.059" rpy="0 0 0" />
     </joint>
     <joint name="left_wheel_joint" type="continuous">
-      <parent link="base_link"/>
-      <child link="left_wheel_link"/>
-      <origin rpy="0 0 0" xyz="0.04025 0.062 -0.024"/>
-      <axis xyz="0 1 0" rpy="0 0 0" />
-      <limit effort="100" velocity="100"/>
-      <dynamics damping="0.5" friction="0.01"/>
+      <parent link="base_link" />
+      <child link="left_wheel_link" />
+      <origin xyz="0.04025 0.062 -0.024" rpy="0 0 0" />
+      <axis xyz="0 1 0" />
+      <limit effort="100" velocity="100" />
+      <dynamics damping="0.5" friction="0.01" />
     </joint>
     <joint name="right_wheel_joint" type="continuous">
-      <parent link="base_link"/>
-      <child link="right_wheel_link"/>
-      <origin rpy="0 0 0" xyz="0.04025 -0.062 -0.024"/>
-      <axis xyz="0 1 0" rpy="0 0 0" />
-      <limit effort="100" velocity="100"/>
-      <dynamics damping="0.5" friction="0.01"/>
+      <parent link="base_link" />
+      <child link="right_wheel_link" />
+      <origin xyz="0.04025 -0.062 -0.024" rpy="0 0 ${-M_PI}" />
+      <axis xyz="0 -1 0" />
+      <limit effort="100" velocity="100" />
+      <dynamics damping="0.5" friction="0.01" />
     </joint>
     <joint name="d435_joint" type="fixed">
-      <parent link="base_link"/>
-      <child link="d435_link"/>
-      <origin rpy="0 0 0" xyz="0.090925 0.0 0.06670"/>
+      <parent link="base_link" />
+      <child link="d435_link" />
+      <origin xyz="0.090925 0.0 0.06670" rpy="0 0 0" />
     </joint>
-     <joint name="lidar_joint" type="fixed">
-      <parent link="base_link"/>
-      <child link="lidar_link"/>
-      <origin rpy="0 0 0" xyz="0.0 0.0 0.125"/>
+    <joint name="lidar_joint" type="fixed">
+      <parent link="base_link" />
+      <child link="lidar_link" />
+      <origin xyz="0.0 0.0 0.125" rpy="0 0 0" />
     </joint>
-    <!--gazebo reference="base_link">
-      <mu1 value="0.0"/>
-      <mu2 value="0.0"/>
-      <kp  value="1000000.0" />
-      <kd  value="1.0" />
-      <fdir1 value="1 0 0"/>
-      <material>Gazebo/White</material>
-      <turnGravityOff>false</turnGravityOff>
-    </gazebo-->
-     <gazebo reference="base_link">
-      <material>Gazebo/White</material>
-      <mu1 value="0.0"/>
-      <mu2 value="0.0"/>
+    <!-- Gazebo Material Assignments
+    <gazebo reference="base_link">
+      <material>Gazebo/Blue</material>
     </gazebo>
     <gazebo reference="left_wheel_link">
-      <mu1 value="3.0"/>
-      <mu2 value="3.0"/>
-      <kp  value="10000000.0" />
-      <kd  value="1.0" />
-      <fdir1 value="1 0 0"/>
       <material>Gazebo/Black</material>
-      <turnGravityOff>false</turnGravityOff>
     </gazebo>
-     <gazebo reference="right_wheel_link">
-      <mu1 value="3.0"/>
-      <mu2 value="3.0"/>
-      <kp  value="10000000.0" />
-      <kd  value="1.0" />
-      <fdir1 value="1 0 0"/>
+    <gazebo reference="right_wheel_link">
       <material>Gazebo/Black</material>
-      <turnGravityOff>false</turnGravityOff>
-    </gazebo>
-    <!-- Transmission is important to link the joints and the controller -->
+    </gazebo>-->
+    <!-- Transmissions -->
     <transmission name="left_wheel_joint_trans">
       <type>transmission_interface/SimpleTransmission</type>
       <joint name="left_wheel_joint" />
       <actuator name="left_wheel_joint_motor">
+        <mechanicalReduction>1</mechanicalReduction>
         <hardwareInterface>EffortJointInterface</hardwareInterface>
-        <mechanicalReduction>1</mechanicalReduction>
       </actuator>
     </transmission>
@@ -162,35 +144,21 @@
       <joint name="right_wheel_joint" />
       <actuator name="right_wheel_joint_motor">
+        <mechanicalReduction>1</mechanicalReduction>
         <hardwareInterface>EffortJointInterface</hardwareInterface>
-        <mechanicalReduction>1</mechanicalReduction>
       </actuator>
     </transmission>
-     <!-- Differential drive controller for Gazebo Ignition -->
-  <gazebo>
-    <plugin filename="gz-sim-diff-drive-system" name="gz::sim::systems::DiffDrive">
-      <!-- wheels -->
-      <left_joint>left_wheel_joint</left_joint>
-      <right_joint>right_wheel_joint</right_joint>
-      <!-- kinematics -->
-      <wheel_separation>${wheel_axle}</wheel_separation>
-      <wheel_radius>${wheel_radius}</wheel_radius>
-      <!-- limits -->
-      <max_linear_acceleration>2</max_linear_acceleration>
-      <max_angular_acceleration>1.5</max_angular_acceleration>
-      <!-- topics -->
-      <topic>cmd_vel</topic>
-      <odom_topic>odom</odom_topic>
-      <tf_topic>tf</tf_topic>
-      <odom_publish_frequency>30</odom_publish_frequency>
-      <frame_id>odom</frame_id>
-      <child_frame_id>base_footprint</child_frame_id>
-    </plugin>
-    <!-- Joint state publisher -->
-    <plugin filename="gz-sim-joint-state-publisher-system" name="gz::sim::systems::JointStatePublisher">
-      <topic>joint_states</topic>
-      <joint_name>left_wheel_joint</joint_name>
-      <joint_name>right_wheel_joint</joint_name>
-    </plugin>
-  </gazebo>
-   </xacro:macro>
+    <!-- Plugin for differential drive control in Gazebo-->
+    <gazebo>
+      <plugin name="ignition::gazebo::systems::DiffDrive" filename="libignition-gazebo-diff-drive-system.so">
+        <left_joint>left_wheel_joint</left_joint>
+        <right_joint>right_wheel_joint</right_joint>
+        <wheel_separation>${wheel_axle}</wheel_separation>
+        <wheel_radius>${wheel_radius}</wheel_radius>
+        <!--<frame_id>base_footprint</frame_id> TO LOOK
+        <ignition_frame_id>base_footprint</ignition_frame_id>-->
+        <odom_publish_frequency>50</odom_publish_frequency>
+        <topic>cmd_vel</topic>
+      </plugin>
+    </gazebo>
+  </xacro:macro>
 </robot>

File: urdf/lidar_gazebo_macro.xacro (robot description, xacro)
@@ -1,63 +1,73 @@
 <?xml version="1.0"?>
-<robot name="lidar_gazebo_macro" xmlns:xacro="http://www.ros.org/wiki/xacro">
-  <!--xacro:include filename="$(find fra2mo_description)/urdf/utility_macro.xacro" /-->
-  <xacro:macro name="lidar_gazebo_sensor" params="parent" >
+<robot xmlns:xacro="http://www.ros.org/wiki/xacro" name="lidar_gazebo_macro" >
+  <!--<xacro:include filename="$(find fra2mo_description)/urdf/utility_macro.xacro" />-->
+  <xacro:macro name="lidar_gazebo_sensor" params="parent">
     <link name="laser_frame">
       <inertial>
-          <inertia ixx="1.0" ixy="0.0" ixz="0.0" iyy="1.0" iyz="0.0" izz="1.0"/>
+        <origin xyz="0 0 0" />
         <mass value="0.1" />
-        <origin xyz="0 0 0" />
-        <cylinder_inertia  m="0.1" r="0.037" h="0.04" />
+        <xacro:cylinder_inertia m="0.1" r="0.037" h="0.04" />
       </inertial>
       <visual>
+        <origin rpy="0 0 ${-M_PI_2}" xyz="0.0 0.0 -0.031" />
         <geometry>
-          <mesh filename="package://fra2mo_description/meshes/lidar.stl" scale="0.001 0.001 0.001 "/>
+          <mesh filename="file://$(find fra2mo_description)/meshes/lidar.stl" scale="0.001 0.001 0.001" />
         </geometry>
-        <material name="White"/>
-        <origin rpy="0 0 ${-M_PI_2}" xyz="0.0 0.0 -0.031"/>
+        <material name="White" />
       </visual>
       <collision>
-        <origin xyz="0 0 0" rpy="0 0 0 " />
+        <origin xyz="0.0 0.0 -0.031" rpy="0 0 0" />
         <geometry>
           <cylinder length="0.04" radius="0.037" />
         </geometry>
-        <origin rpy="0 0 0" xyz="0.0 0.0 -0.031"/>
       </collision>
     </link>
     <joint name="laser_joint" type="fixed">
-      <parent link="${parent}"/>
-      <child link="laser_frame"/>
-      <origin rpy="0 0 0" xyz="0.0 0.0 0.031"/>
+      <parent link="${parent}" />
+      <child link="laser_frame" />
+      <origin rpy="0 0 0" xyz="0.0 0.0 0.031" />
     </joint>
     <gazebo reference="laser_frame">
-      <sensor type="gpu_lidar" name="head_hokuyo_sensor">
-        <pose>0 0 0 0 0 0</pose>
-        <visualize>false</visualize>
-        <update_rate>40</update_rate>
-        <topic>scan</topic>
-        <gz_frame_id>laser_frame</gz_frame_id>
-        <lidar>
-            <scan>
-              <horizontal>
-                <samples>720</samples>
-                <resolution>1</resolution>
-                <min_angle>-${M_PI}</min_angle>
-                <max_angle>${M_PI}</max_angle>
-              </horizontal>
-            </scan>
-            <range>
-              <min>0.8</min>
-              <max>30.0</max>
-              <resolution>0.01</resolution>
-            </range>
-            <noise>
-              <type>gaussian</type>
-              <mean>0.0</mean>
-              <stddev>0.01</stddev>
-            </noise>
-        </lidar>
-        <always_on>true</always_on>
-      </sensor>
+      <sensor name="laser_frame" type="gpu_lidar">
+          <!--<pose relative_to="laser_frame">0 0 0 0 0 0</pose>--> <!--TO LOOK-->
+          <topic>lidar</topic>
+          <update_rate>10</update_rate>
+          <ray>
+              <scan>
+                  <horizontal>
+                      <samples>640</samples>
+                      <resolution>1</resolution>
+                      <min_angle>-3.14</min_angle>
+                      <max_angle>3.14</max_angle>
+                  </horizontal>
+                  <!--<vertical>
+                      <samples>640</samples>
+                      <resolution>1</resolution>
+                      <min_angle>-1.61799</min_angle>
+                      <max_angle>1.661799</max_angle>
+                  </vertical>-->
+              </scan>
+              <range>
+                  <min>0.1</min>
+                  <max>10.0</max>
+                  <resolution>0.01</resolution>
+              </range>
+            </ray>
+            <always_on>false</always_on>
+            <visualize>false</visualize>
+            <frame_id>laser_frame</frame_id> <!--TO LOOK-->
+            <ignition_frame_id>laser_frame</ignition_frame_id>
+        </sensor>
     </gazebo>
+  <!--TO LOOK-->
+  <!--<gazebo>
+    <plugin filename="libignition-gazebo-sensors-system.so"
+      name="ignition::gazebo::systems::Sensors">
+        <render_engine>ogre2</render_engine>
+    </plugin>
+  </gazebo>-->
+  <gazebo>
+  <plugin filename="ignition-gazebo-sensors-system" name="gz::sim::systems::Sensors" />
+  </gazebo>
   </xacro:macro>
 </robot>
