Commit message: Salva ultime modifiche, aggiorna urdf, rimuovi test.urdf e meshes copy, aggiungi nuove mesh

File: urdf/d435_gazebo_macro.xacro (robot description, xacro)
@@ -7,8 +7,10 @@
     </xacro:sensor_d435>
     <gazebo reference="${parent}">
-      <sensor type="depth_camera" name="depth_camera">
+      <sensor type="rgbd_camera" name="depth_camera">
         <always_on>true</always_on>
         <update_rate>30.0</update_rate>
-        <camera>
+        <topic>depth_camera</topic>
+        <gz_frame_id>d435_link</gz_frame_id>
+        <ignition_frame_id>d435_link</ignition_frame_id> <camera>
           <horizontal_fov>1.3962634</horizontal_fov>
           <image>
@@ -18,19 +20,8 @@
           </image>
           <clip>
-            <near>0.01</near>
-            <far>100</far>
+            <near>0.1</near>
+            <far>30</far>
           </clip>
         </camera>
-        <plugin name="GazeboRosDepthCamera" filename="libgazebo_ros_depth_camera.so">
-          <ros>
-            <namespace>/</namespace>
-            <remapping>~/depth/image_raw:=/depth_camera/image_raw</remapping>
-            <remapping>~/depth/camera_info:=/depth_camera/camera_info</remapping>
-            <remapping>~/points:=/depth/points</remapping>
-          </ros>
-          <update_rate>30.0</update_rate>
-          <camera_name>depth_camera</camera_name>
-          <frame_name>camera_depth_optical_frame</frame_name>
-        </plugin>
       </sensor>
     </gazebo>

File: urdf/fra2mo_base_macro.xacro (robot description, xacro)
@@ -4,4 +4,6 @@
   <!-- WHOLE BASE MACRO-->
   <xacro:macro name="fra2mo_base" > <!--fb : front, back ; lr: left, right -->
+  <!-- Odometry root frame -->
+  <link name="base_footprint"/>
     <!-- Base properties -->
     <xacro:property name="base_height" value="0.180" />
@@ -11,7 +13,4 @@
     <xacro:property name="wheel_radius" value="0.035" />
     <xacro:property name="wheel_axle" value="0.13" />
-    <!-- Actual body/chassis of the robot -->
-    <link name="base_footprint">
-    </link>
     <link name="base_link">
       <!-- Inertial properties -->
@@ -54,7 +53,7 @@
       <collision>
         <geometry>
-          <mesh filename="file://$(find fra2mo_description)/meshes/fra2mo_wheel.stl" scale="0.001 0.001 0.001" />
+          <cylinder length="0.02" radius="${wheel_radius}" />
         </geometry>
-        <origin xyz="0 0 0" rpy="0 0 0" />
+        <origin xyz="0 0 0" rpy="0 1.5708 1.5708" />
       </collision>
       <inertial>
@@ -75,7 +74,7 @@
       <collision>
         <geometry>
-          <mesh filename="file://$(find fra2mo_description)/meshes/fra2mo_wheel.stl" scale="0.001 0.001 0.001" />
+          <cylinder length="0.02" radius="${wheel_radius}" />
         </geometry>
-        <origin xyz="0 0 0" rpy="0 0 0" />
+        <origin xyz="0 0 0" rpy="0 1.5708 1.5708" />
       </collision>
       <inertial>
@@ -150,13 +149,24 @@
     <!-- Plugin for differential drive control in Gazebo-->
     <gazebo>
-      <plugin name="ignition::gazebo::systems::DiffDrive" filename="libignition-gazebo-diff-drive-system.so">
+      <plugin filename="libignition-gazebo-diff-drive-system.so" name="ignition::gazebo::systems::DiffDrive">
         <left_joint>left_wheel_joint</left_joint>
         <right_joint>right_wheel_joint</right_joint>
         <wheel_separation>${wheel_axle}</wheel_separation>
         <wheel_radius>${wheel_radius}</wheel_radius>
-        <!--<frame_id>base_footprint</frame_id> TO LOOK
-        <ignition_frame_id>base_footprint</ignition_frame_id>-->
+        <max_linear_acceleration>1.0</max_linear_acceleration>
+        <min_linear_acceleration>-1.0</min_linear_acceleration>
+        <max_angular_acceleration>1.0</max_angular_acceleration>
+        <min_angular_acceleration>-1.0</min_angular_acceleration>
+        <max_linear_velocity>2.0</max_linear_velocity>
+        <min_linear_velocity>-2.0</min_linear_velocity>
+        <max_angular_velocity>2.0</max_angular_velocity>
+        <min_angular_velocity>-2.0</min_angular_velocity>
+        <frame_id>odom</frame_id>
+        <child_frame_id>base_footprint</child_frame_id>
         <odom_publish_frequency>50</odom_publish_frequency>
+        <odom_topic>odom</odom_topic>
         <topic>cmd_vel</topic>
+        <publish_odom>true</publish_odom>
+        <publish_odom_tf>true</publish_odom_tf>
       </plugin>
     </gazebo>

File: urdf/lidar_gazebo_macro.xacro (robot description, xacro)
@@ -29,33 +29,35 @@
     </joint>
     <gazebo reference="laser_frame">
-      <sensor name="laser_frame" type="gpu_lidar">
-          <!--<pose relative_to="laser_frame">0 0 0 0 0 0</pose>--> <!--TO LOOK-->
-          <topic>lidar</topic>
+        <sensor name="laser_frame" type="gpu_lidar">
+          <topic>scan</topic>
           <update_rate>10</update_rate>
           <ray>
-              <scan>
-                  <horizontal>
-                      <samples>640</samples>
-                      <resolution>1</resolution>
-                      <min_angle>-3.14</min_angle>
-                      <max_angle>3.14</max_angle>
-                  </horizontal>
-                  <!--<vertical>
-                      <samples>640</samples>
-                      <resolution>1</resolution>
-                      <min_angle>-1.61799</min_angle>
-                      <max_angle>1.661799</max_angle>
-                  </vertical>-->
-              </scan>
-              <range>
-                  <min>0.1</min>
-                  <max>10.0</max>
-                  <resolution>0.01</resolution>
-              </range>
-            </ray>
-            <always_on>false</always_on>
-            <visualize>false</visualize>
-            <frame_id>laser_frame</frame_id> <!--TO LOOK-->
-            <ignition_frame_id>laser_frame</ignition_frame_id>
+            <scan>
+              <horizontal>
+                <samples>640</samples>
+                <resolution>1</resolution>
+                <min_angle>-3.14</min_angle>
+                <max_angle>3.14</max_angle>
+              </horizontal>
+            </scan>
+            <range>
+              <min>0.1</min>
+              <max>10.0</max>
+              <resolution>0.01</resolution>
+            </range>
+          </ray>
+          <always_on>true</always_on>
+          <visualize>true</visualize>
+          <frame_id>laser_frame</frame_id>
+          <ignition_frame_id>laser_frame</ignition_frame_id>
+          <!-- Plugin ROS classic per pubblicare su topic ROS
+          <plugin name="gazebo_ros_laser" filename="libgazebo_ros_ray_sensor.so">
+            <ros>
+            <namespace>/</namespace>
+            <remapping>~/scan:=/scan</remapping>
+            </ros>
+            <frame_name>laser_frame</frame_name>
+            <topic>scan</topic>
+          </plugin>-->
         </sensor>
     </gazebo>

Commit message: Update files

File: urdf/d435_gazebo_macro.xacro (robot description, xacro)
@@ -6,11 +6,14 @@
       <origin xyz="0 0 0" rpy="0 0 0" />
     </xacro:sensor_d435>
+    <!--The following code adds a Gazebo plugin to the camera sensor,
+    which allows it to publish depth images in the Gazebo simulation environment.-->
     <gazebo reference="${parent}">
       <sensor type="rgbd_camera" name="depth_camera">
         <always_on>true</always_on>
         <update_rate>30.0</update_rate>
+        <!--Topic name of camera-->
         <topic>depth_camera</topic>
-        <gz_frame_id>d435_link</gz_frame_id>
-        <ignition_frame_id>d435_link</ignition_frame_id> <camera>
+        <!--Frame ID of the camera-->
+        <gz_frame_id>d435_link</gz_frame_id><camera>
           <horizontal_fov>1.3962634</horizontal_fov>
           <image>

File: urdf/fra2mo.urdf.xacro (robot description, xacro)
@@ -1,3 +1,5 @@
 <?xml version="1.0"?>
+<!--This file defines the URDF for the Fra2Mo robot,
+ including its base, LIDAR, and RGBD sensors.-->
 <robot xmlns:xacro="http://www.ros.org/wiki/xacro" name="fra2mo" >
   <xacro:include filename="$(find fra2mo_description)/urdf/fra2mo_base_macro.xacro"/>

File: urdf/fra2mo_base_macro.xacro (robot description, xacro)
@@ -2,6 +2,5 @@
 <robot  xmlns:xacro="http://www.ros.org/wiki/xacro">
   <xacro:include filename="$(find fra2mo_description)/urdf/utility_macro.xacro" />
-  <!-- WHOLE BASE MACRO-->
-  <xacro:macro name="fra2mo_base" > <!--fb : front, back ; lr: left, right -->
+  <xacro:macro name="fra2mo_base" >
   <!-- Odometry root frame -->
   <link name="base_footprint"/>
@@ -120,15 +119,5 @@
       <origin xyz="0.0 0.0 0.125" rpy="0 0 0" />
     </joint>
-    <!-- Gazebo Material Assignments
-    <gazebo reference="base_link">
-      <material>Gazebo/Blue</material>
-    </gazebo>
-    <gazebo reference="left_wheel_link">
-      <material>Gazebo/Black</material>
-    </gazebo>
-    <gazebo reference="right_wheel_link">
-      <material>Gazebo/Black</material>
-    </gazebo>-->
-    <!-- Transmissions -->
+    <!-- Transmissions for the wheel joints -->
     <transmission name="left_wheel_joint_trans">
       <type>transmission_interface/SimpleTransmission</type>
@@ -156,4 +145,5 @@
         <wheel_separation>${wheel_axle}</wheel_separation>
         <wheel_radius>${wheel_radius}</wheel_radius>
+        <!-- Limits for the differential drive -->
         <max_linear_acceleration>1.0</max_linear_acceleration>
         <min_linear_acceleration>-1.0</min_linear_acceleration>
@@ -166,4 +156,5 @@
         <odom_publish_frequency>50</odom_publish_frequency>
         <topic>/cmd_vel</topic>
+        <!-- Odometry and TF topics -->
         <odom_topic>/odom</odom_topic>
         <tf_topic>/tf</tf_topic>
@@ -174,4 +165,5 @@
         <publish_wheel_tf>true</publish_wheel_tf>
       </plugin>
+      <!-- Joint State Publisher plugin -->
       <plugin
         filename="libgz-sim-joint-state-publisher-system.so"

File: urdf/lidar_gazebo_macro.xacro (robot description, xacro)
@@ -1,6 +1,7 @@
 <?xml version="1.0"?>
 <robot xmlns:xacro="http://www.ros.org/wiki/xacro" name="lidar_gazebo_macro" >
-  <!--<xacro:include filename="$(find fra2mo_description)/urdf/utility_macro.xacro" />-->
+  <!--xacro:include filename="$(find fra2mo_description)/urdf/utility_macro.xacro" /-->
   <xacro:macro name="lidar_gazebo_sensor" params="parent">
+    <!-- Lidar is composed by a single link and a fixed joint -->
     <link name="laser_frame">
       <inertial>
@@ -28,8 +29,11 @@
       <origin rpy="0 0 0" xyz="0.0 0.0 0.031" />
     </joint>
+    <!-- Gazebo plugin for the LiDAR sensor -->
     <gazebo reference="laser_frame">
       <sensor name="lidar" type="gpu_lidar">
+        <!-- Frame ID for the LiDAR sensor -->
         <gz_frame_id>laser_frame</gz_frame_id>
         <pose>0 0 0 0 0 0</pose>
+        <!-- Topic name for the LiDAR data -->
         <topic>/scan</topic>
         <update_rate>10</update_rate>
@@ -53,4 +57,5 @@
       </sensor>
     </gazebo>
+    <!-- Gazebo plugin for the LiDAR sensor -->
     <gazebo>
     <plugin
