Commit message: Aggiorna fra2mo_conf_ros2.rviz e fra2mo_base_macro.xacro

File: urdf/fra2mo_base_macro.xacro (robot description, xacro)
@@ -5,8 +5,8 @@
 	<xacro:property name="base_height" value="0.180" />
   <xacro:property name="base_radius" value="0.11" />
-  <xacro:property name="base_mass" value="5" />
-  <xacro:property name="wheel_mass" value="2.5" />
+  <xacro:property name="base_mass" value="2" />
+  <xacro:property name="wheel_mass" value="0.2" />
   <xacro:property name="wheel_radius" value="0.035" />
-  <xacro:property name="wheel_axle" value="0.130" />
+  <xacro:property name="wheel_axle" value="0.124" />
   <!-- WHOLE BASE MACRO-->
   <xacro:macro name="fra2mo_base" > <!--fb : front, back ; lr: left, right -->
@@ -16,8 +16,7 @@
     <link name="base_link">
       <inertial>
-          <inertia ixx="1.0" ixy="0.0" ixz="0.0" iyy="1.0" iyz="0.0" izz="1.0"/>
         <mass value="${base_mass}" />
-        <origin xyz="0 0 0" />
-        <cylinder_inertia  m="${base_mass}" r="${base_radius}" h="${base_height}" />
+        <origin xyz="0 0 -0.05" /> <!-- baricentro abbassato di 5 cm -->
+        <inertia ixx="0.01145" ixy="0.0" ixz="0.0" iyy="0.01145" iyz="0.0" izz="0.0121"/>
       </inertial>
       <visual>
@@ -51,14 +50,13 @@
       <collision>
         <geometry>
-          <mesh filename="package://fra2mo_description/meshes/fra2mo_wheel.stl" scale="0.001 0.001 0.001 "/>
-        </geometry>
-        <origin rpy="0 0 0" xyz="0 0 0"/>
+          <cylinder radius="${wheel_radius}" length="0.02"/> </geometry>
+        <origin rpy="1.570796 0 0" xyz="0 0 0"/>
       </collision>
       <inertial>
-        <mass value="${wheel_mass}" />
-        <origin xyz="0 0 0" />
-        <inertia ixx="0.001" ixy="0.0" ixz="0.0"
-               iyy="0.001" iyz="0.0"
-               izz="0.001" />
+          <mass value="${wheel_mass}" />
+          <origin xyz="0 0 0" />
+          <inertia ixx="0.0000679" ixy="0.0" ixz="0.0"
+                   iyy="0.0000679" iyz="0.0"
+                   izz="0.0001225" />
       </inertial>
     </link>
@@ -73,14 +71,13 @@
       <collision>
         <geometry>
-          <mesh filename="package://fra2mo_description/meshes/fra2mo_wheel.stl" scale="0.001 0.001 0.001 "/>
-        </geometry>
-        <origin rpy="0 0 0" xyz="0 0 0"/>
+          <cylinder radius="${wheel_radius}" length="0.02"/> </geometry>
+        <origin rpy="1.570796 0 0" xyz="0 0 0"/>
       </collision>
       <inertial>
-        <mass value="${wheel_mass}" />
-        <origin xyz="0 0 0" />
-        <inertia ixx="0.001" ixy="0.0" ixz="0.0"
-               iyy="0.001" iyz="0.0"
-               izz="0.001" />
+          <mass value="${wheel_mass}" />
+          <origin xyz="0 0 0" />
+          <inertia ixx="0.0000679" ixy="0.0" ixz="0.0"
+                   iyy="0.0000679" iyz="0.0"
+                   izz="0.0001225" />
       </inertial>
     </link>
@@ -100,13 +97,13 @@
       <axis xyz="0 1 0" rpy="0 0 0" />
       <limit effort="100" velocity="100"/>
-      <joint_properties damping="0.5" friction="0.01"/>
+      <dynamics damping="0.5" friction="0.01"/>
     </joint>
     <joint name="right_wheel_joint" type="continuous">
       <parent link="base_link"/>
       <child link="right_wheel_link"/>
-      <origin rpy="0 0 ${-M_PI}" xyz="0.04025 -0.062 -0.024"/>
-      <axis xyz="0 -1 0" rpy="0 0 0" />
+      <origin rpy="0 0 0" xyz="0.04025 -0.062 -0.024"/>
+      <axis xyz="0 1 0" rpy="0 0 0" />
       <limit effort="100" velocity="100"/>
-      <joint_properties damping="0.5" friction="0.01"/>
+      <dynamics damping="0.5" friction="0.01"/>
     </joint>
     <joint name="d435_joint" type="fixed">
@@ -131,9 +128,11 @@
      <gazebo reference="base_link">
       <material>Gazebo/White</material>
+      <mu1 value="0.0"/>
+      <mu2 value="0.0"/>
     </gazebo>
     <gazebo reference="left_wheel_link">
-      <mu1 value="1.0"/>
-      <mu2 value="1.0"/>
-      <kp  value="1000000.0" />
+      <mu1 value="3.0"/>
+      <mu2 value="3.0"/>
+      <kp  value="10000000.0" />
       <kd  value="1.0" />
       <fdir1 value="1 0 0"/>
@@ -142,7 +141,7 @@
     </gazebo>
      <gazebo reference="right_wheel_link">
-      <mu1 value="1.0"/>
-      <mu2 value="1.0"/>
-      <kp  value="1000000.0" />
+      <mu1 value="3.0"/>
+      <mu2 value="3.0"/>
+      <kp  value="10000000.0" />
       <kd  value="1.0" />
       <fdir1 value="1 0 0"/>
@@ -177,11 +176,11 @@
       <wheel_radius>${wheel_radius}</wheel_radius>
       <!-- limits -->
-      <max_linear_acceleration>1.0</max_linear_acceleration>
-      <max_angular_acceleration>2.0</max_angular_acceleration>
+      <max_linear_acceleration>2</max_linear_acceleration>
+      <max_angular_acceleration>1.5</max_angular_acceleration>
       <!-- topics -->
       <topic>cmd_vel</topic>
       <odom_topic>odom</odom_topic>
       <tf_topic>tf</tf_topic>
-      <odom_publish_frequency>50</odom_publish_frequency>
+      <odom_publish_frequency>30</odom_publish_frequency>
       <frame_id>odom</frame_id>
       <child_frame_id>base_footprint</child_frame_id>

Commit message: Update FRA2MO description assets and base macro

File: urdf/fra2mo_base_macro.xacro (robot description, xacro)
@@ -118,5 +118,5 @@
       <parent link="base_link" />
       <child link="lidar_link" />
-      <origin xyz="0.0 0.0 0.125" rpy="0 0 0" />
+      <origin xyz="0.0 0.0 0.125" rpy="0 0 ${M_PI}" />
     </joint>
     <transmission name="left_wheel_joint_trans">
